Commit message: links for meshes

File: install/KR600_2830_description/share/KR600_2830_description/urdf/model.urdf (robot description, URDF)
Before this commit: robot KR600_R2830, 7 links, 6 joints
Links:
- link base_link: geometry collision mesh filename=meshes/base_link.stl scale=0.001 0.001 0.001; visual mesh filename=meshes/base_link.stl scale=0.001 0.001 0.001
- link link1: geometry collision mesh filename=meshes/link1.stl scale=0.001 0.001 0.001; visual mesh filename=meshes/link1.stl scale=0.001 0.001 0.001
- link link2: geometry collision mesh filename=meshes/link2.stl scale=0.001 0.001 0.001; visual mesh filename=meshes/link2.stl scale=0.001 0.001 0.001
- link link3: geometry collision mesh filename=meshes/link3.stl scale=0.001 0.001 0.001; visual mesh filename=meshes/link3.stl scale=0.001 0.001 0.001
- link link4: geometry collision mesh filename=meshes/link4.stl scale=0.001 0.001 0.001; visual mesh filename=meshes/link4.stl scale=0.001 0.001 0.001
- link link5: geometry collision mesh filename=meshes/link5.stl scale=0.001 0.001 0.001; visual mesh filename=meshes/link5.stl scale=0.001 0.001 0.001
- link link6: geometry collision mesh filename=meshes/link6.stl scale=0.001 0.001 0.001; visual mesh filename=meshes/link6.stl scale=0.001 0.001 0.001
