Commit message: update

File: install/kr600/share/kr600/urdf/model.urdf.xacro (robot description, xacro)
@@ -1,9 +1,19 @@
 <?xml version="1.0" ?>
 <robot xmlns:xacro="http://wiki.ros.org/xacro" name="kr600">
+ <xacro:property name="mesh_path" value="../meshes"/>
 <link name="base_link">
+        <inertial>
+            <origin xyz="0 0 0" rpy="0 0 0"/>
+            <mass value="1.0"/> <!-- Заменить на фактическую массу -->
+            <inertia ixx="0.1" ixy="0.0" ixz="0.0" iyy="0.1" iyz="0.0" izz="0.1"/> <!-- Заменить на фактические моменты инерции -->
+        </inertial>
         <visual name="base_link_visual">
             <origin xyz="0.0 0.0 0.0" rpy="0.0 0.0 0.0" />
             <geometry>
-                <mesh filename="package://kr600/meshes/base_link.stl" scale="0.001 0.001 0.001" />
+<!--                                               $ (find kr600)/meshes/base_link.stl   -->
+<!-- /root/dream_ws/install/kr600/share/kr600/urdf/$(find kr600)/meshes/base_link.stl   -->
+<!-- /root/dream_ws/install/kr600/share/kr600/urdf/$ (find kr600)/meshes/base_link.stl   -->
+<!-- package:/ -->
+                <mesh filename="../meshes/base_link.stl" scale="0.001 0.001 0.001" />
             </geometry>
         </visual>
@@ -11,5 +21,5 @@
             <origin xyz="0.0 0.0 0.0" rpy="0.0 0.0 0.0" />
             <geometry>
-                <mesh filename="package://kr600/meshes/base_link.stl" scale="0.001 0.001 0.001" />
+                <mesh filename="../meshes/base_link.stl" scale="0.001 0.001 0.001" />
             </geometry>
         </collision>
@@ -24,5 +34,5 @@
             <origin xyz="6.93889390390723e-18 0.0 0.556" rpy="3.141592653589793 -0.0 0.0" />
             <geometry>
-                <mesh filename="package://kr600/meshes/link1.stl" scale="0.001 0.001 0.001" />
+                <mesh filename="../meshes/link1.stl" scale="0.001 0.001 0.001" />
             </geometry>
         </visual>
@@ -30,5 +40,5 @@
             <origin xyz="6.93889390390723e-18 0.0 0.556" rpy="3.141592653589793 -0.0 0.0" />
             <geometry>
-                <mesh filename="package://kr600/meshes/link1.stl" scale="0.001 0.001 0.001" />
+                <mesh filename="../meshes/link1.stl" scale="0.001 0.001 0.001" />
             </geometry>
         </collision>
@@ -43,5 +53,5 @@
             <origin xyz="-0.5 -1.045 -0.054000000000000006" rpy="-1.5707963267948966 -0.0 0.0" />
             <geometry>
-                <mesh filename="package://kr600/meshes/link2.stl" scale="0.001 0.001 0.001" />
+                <mesh filename="../meshes/link2.stl" scale="0.001 0.001 0.001" />
             </geometry>
         </visual>
@@ -49,5 +59,5 @@
             <origin xyz="-0.5 -1.045 -0.054000000000000006" rpy="-1.5707963267948966 -0.0 0.0" />
             <geometry>
-                <mesh filename="package://kr600/meshes/link2.stl" scale="0.001 0.001 0.001" />
+                <mesh filename="../meshes/link2.stl" scale="0.001 0.001 0.001" />
             </geometry>
         </collision>
@@ -62,5 +72,5 @@
             <origin xyz="-0.500000000000006 2.345 0.255" rpy="1.5707963267948966 -0.0 0.0" />
             <geometry>
-                <mesh filename="package://kr600/meshes/link3.stl" scale="0.001 0.001 0.001" />
+                <mesh filename="../meshes/link3.stl" scale="0.001 0.001 0.001" />
             </geometry>
         </visual>
@@ -68,5 +78,5 @@
             <origin xyz="-0.500000000000006 2.345 0.255" rpy="1.5707963267948966 -0.0 0.0" />
             <geometry>
-                <mesh filename="package://kr600/meshes/link3.stl" scale="0.001 0.001 0.001" />
+                <mesh filename="../meshes/link3.stl" scale="0.001 0.001 0.001" />
             </geometry>
         </collision>
@@ -81,5 +91,5 @@
             <origin xyz="-2.29 0.0 0.9890000000000061" rpy="-0.0 1.5707963267948966 0" />
             <geometry>
-                <mesh filename="package://kr600/meshes/link4.stl" scale="0.001 0.001 0.001" />
+                <mesh filename="../meshes/link4.stl" scale="0.001 0.001 0.001" />
             </geometry>
         </visual>
@@ -87,5 +97,5 @@
             <origin xyz="-2.29 0.0 0.9890000000000061" rpy="-0.0 1.5707963267948966 0" />
             <geometry>
-                <mesh filename="package://kr600/meshes/link4.stl" scale="0.001 0.001 0.001" />
+                <mesh filename="../meshes/link4.stl" scale="0.001 0.001 0.001" />
             </geometry>
         </collision>
@@ -100,5 +110,5 @@
             <origin xyz="-1.525000000000006 2.29 -0.17500000000000002" rpy="1.5707963267948966 -0.0 0.0" />
             <geometry>
-                <mesh filename="package://kr600/meshes/link5.stl" scale="0.001 0.001 0.001" />
+                <mesh filename="../meshes/link5.stl" scale="0.001 0.001 0.001" />
             </geometry>
         </visual>
@@ -106,5 +116,5 @@
             <origin xyz="-1.525000000000006 2.29 -0.17500000000000002" rpy="1.5707963267948966 -0.0 0.0" />
             <geometry>
-                <mesh filename="package://kr600/meshes/link5.stl" scale="0.001 0.001 0.001" />
+                <mesh filename="../meshes/link5.stl" scale="0.001 0.001 0.001" />
             </geometry>
         </collision>
@@ -119,5 +129,5 @@
             <origin xyz="-2.29 0.0 -1.7620000000000058" rpy="-3.141592653589793 -1.5707963267948966 0" />
             <geometry>
-                <mesh filename="package://kr600/meshes/link6.stl" scale="0.001 0.001 0.001" />
+                <mesh filename="../meshes/link6.stl" scale="0.001 0.001 0.001" />
             </geometry>
         </visual>
@@ -125,5 +135,5 @@
             <origin xyz="-2.29 0.0 -1.7620000000000058" rpy="-3.141592653589793 -1.5707963267948966 0" />
             <geometry>
-                <mesh filename="package://kr600/meshes/link6.stl" scale="0.001 0.001 0.001" />
+                <mesh filename="../meshes/link6.stl" scale="0.001 0.001 0.001" />
             </geometry>
         </collision>
@@ -165,3 +175,7 @@
         <axis xyz="0.0 0.0 1.0" />
     </joint>
+    <!--=================== GAZEBO ================-->
+    <gazebo reference="base_link">
+        <fixed >true</fixed >
+    </gazebo>
 </robot>

Commit message: materials

File: install/kr600/share/kr600/urdf/model.urdf.xacro (robot description, xacro)
@@ -1,5 +1,6 @@
 <?xml version="1.0" ?>
 <robot xmlns:xacro="http://wiki.ros.org/xacro" name="kr600">
- <xacro:property name="mesh_path" value="../meshes"/>
+<xacro:property name="mesh_path" value="../meshes"/>
+<link name="world"></link>
 <link name="base_link">
         <inertial>
@@ -11,10 +12,7 @@
             <origin xyz="0.0 0.0 0.0" rpy="0.0 0.0 0.0" />
             <geometry>
-<!--                                               $ (find kr600)/meshes/base_link.stl   -->
-<!-- /root/dream_ws/install/kr600/share/kr600/urdf/$(find kr600)/meshes/base_link.stl   -->
-<!-- /root/dream_ws/install/kr600/share/kr600/urdf/$ (find kr600)/meshes/base_link.stl   -->
-<!-- package:/ -->
                 <mesh filename="../meshes/base_link.stl" scale="0.001 0.001 0.001" />
             </geometry>
+            <material name="Orange1"/>
         </visual>
         <collision name="base_link_collision">
@@ -36,4 +34,5 @@
                 <mesh filename="../meshes/link1.stl" scale="0.001 0.001 0.001" />
             </geometry>
+            <material name="Black"/>
         </visual>
         <collision name="link1_collision">
@@ -55,4 +54,5 @@
                 <mesh filename="../meshes/link2.stl" scale="0.001 0.001 0.001" />
             </geometry>
+            <material name="Orange2"/>
         </visual>
         <collision name="link2_collision">
@@ -74,4 +74,5 @@
                 <mesh filename="../meshes/link3.stl" scale="0.001 0.001 0.001" />
             </geometry>
+            <material name="Orange2"/>
         </visual>
         <collision name="link3_collision">
@@ -93,4 +94,5 @@
                 <mesh filename="../meshes/link4.stl" scale="0.001 0.001 0.001" />
             </geometry>
+            <material name="Orange2"/>
         </visual>
         <collision name="link4_collision">
@@ -112,4 +114,5 @@
                 <mesh filename="../meshes/link5.stl" scale="0.001 0.001 0.001" />
             </geometry>
+            <material name="Orange1"/>
         </visual>
         <collision name="link5_collision">
@@ -131,4 +134,5 @@
                 <mesh filename="../meshes/link6.stl" scale="0.001 0.001 0.001" />
             </geometry>
+            <material name="Black"/>
         </visual>
         <collision name="link6_collision">
@@ -139,4 +143,10 @@
         </collision>
     </link>
+    <!--======================= JOINTS =========================-->
+    <joint name="world__base_link" type="fixed">
+        <parent link="world"/>
+        <child link="base_link"/>
+        <origin xyz="0.0 0.0 0.0" rpy="0.0 0.0 0.0"/>
+    </joint>
     <joint name="base_link_joint_base_link__link1" type="continuous">
         <origin xyz="0.0 0.0 0.5660000000000001" rpy="3.141592653589793 -0.0 0.0" />
@@ -176,6 +186,12 @@
     </joint>
     <!--=================== GAZEBO ================-->
-    <gazebo reference="base_link">
-        <fixed >true</fixed >
-    </gazebo>
+    <material name="Orange1">
+        <color rgba="1.0 0.1 0.0 1.0"/>
+    </material>
+    <material name="Orange2">
+        <color rgba="1.0 0.15 0.1 1.0"/>
+    </material>
+    <material name="Black">
+        <color rgba="0.1 0.1 0.1 1.0"/>
+    </material>
 </robot>
