Commit message: robot table

File: src/kr600/urdf/model.urdf.xacro (robot description, xacro)
@@ -2,13 +2,37 @@
 <robot xmlns:xacro="http://wiki.ros.org/xacro" name="kr600">
 <xacro:property name="mesh_path" value="../meshes"/>
-<link name="world"></link>
-<link name="base_link">
-        <inertial>
-            <origin xyz="0 0 0" rpy="0 0 0"/>
-            <mass value="1.0"/> <!-- Заменить на фактическую массу -->
-            <inertia ixx="0.1" ixy="0.0" ixz="0.0" iyy="0.1" iyz="0.0" izz="0.1"/> <!-- Заменить на фактические моменты инерции -->
+   <!-- ===================== JOINTS ============================ -->
+    <link name="world">
+    </link>
+    <link name="table">
+        <inertial>
+            <origin xyz="0.0 0.0 0.6" rpy="0.0 0.0 0.0" />
+            <mass value="11455.191000000003" />
+            <inertia ixx="2543.468607273" iyy="2543.468607273" izz="2310.1301850000045" ixy="-1.4972686767578125e-12" iyz="0.0" ixz="0.0" />
+        </inertial>
+        <visual name="table_visual">
+            <origin xyz="0.0 0.0 0.6" rpy="0.0 0.0 0.0" />
+            <geometry>
+                <box size="1.1 1.1 1.2" scale="0.001 0.001 0.001"/>
+                <!-- <mesh filename="../meshes/table.stl" scale="0.001 0.001 0.001" />> -->
+            </geometry>
+            <material name="Black"/>
+        </visual>
+        <collision name="table_collision">
+            <origin xyz="0.0 0.0 0.6" rpy="0.0 0.0 0.0" />
+            <geometry>
+                <box size="1.1 1.1 1.2" scale="0.001 0.001 0.001"/>
+                <!-- <mesh filename="../meshes/table.stl" scale="0.001 0.001 0.001" /> -->
+            </geometry>
+        </collision>
+    </link>
+    <link name="base_link">
+        <inertial>
+            <origin xyz="-0.020452383481017185 -2.2516300426230943e-05 0.2834119414959318" rpy="0.0 -0.0 0.0" />
+            <mass value="2776.5227672504325" />
+            <inertia ixx="207.7193498156812" iyy="234.02781059843255" izz="299.3121468379332" ixy="-0.10431058436127894" iyz="-0.0009718611617845901" ixz="2.078775166299863" />
         </inertial>
         <visual name="base_link_visual">
-            <origin xyz="0.0 0.0 0.0" rpy="0.0 0.0 0.0" />
+            <origin xyz="0.0 0.0 -0.005999999999999943" rpy="0.0 -0.0 0.0" />
             <geometry>
                 <mesh filename="../meshes/base_link.stl" scale="0.001 0.001 0.001" />
@@ -17,5 +41,5 @@
         </visual>
         <collision name="base_link_collision">
-            <origin xyz="0.0 0.0 0.0" rpy="0.0 0.0 0.0" />
+            <origin xyz="0.0 0.0 -0.005999999999999943" rpy="0.0 -0.0 0.0" />
             <geometry>
                 <mesh filename="../meshes/base_link.stl" scale="0.001 0.001 0.001" />
@@ -25,10 +49,10 @@
     <link name="link1">
         <inertial>
-            <origin xyz="0.07579150865291566 0.00268206936456012 -0.27274381273616777" rpy="0.0 -0.0 0.0" />
+            <origin xyz="0.07579150865291566 0.00268206936456012 -0.272743812736168" rpy="0.0 -0.0 0.0" />
             <mass value="1646.969281489809" />
-            <inertia ixx="98.17307546872144" iyy="186.2249092649879" izz="188.8400824035311" ixy="32.477007978946276" iyz="1.1729243360083919" ixz="31.338405874445556" />
+            <inertia ixx="98.17307546872144" iyy="186.22490926498813" izz="188.8400824035311" ixy="32.477007978946276" iyz="1.1729243360083927" ixz="31.3384058744455" />
         </inertial>
         <visual name="link1_visual">
-            <origin xyz="6.93889390390723e-18 0.0 0.556" rpy="3.141592653589793 -0.0 0.0" />
+            <origin xyz="6.661338147750939e-18 0.0 0.5559999999999999" rpy="3.141592653589793 -0.0 0.0" />
             <geometry>
                 <mesh filename="../meshes/link1.stl" scale="0.001 0.001 0.001" />
@@ -37,5 +61,5 @@
         </visual>
         <collision name="link1_collision">
-            <origin xyz="6.93889390390723e-18 0.0 0.556" rpy="3.141592653589793 -0.0 0.0" />
+            <origin xyz="6.661338147750939e-18 0.0 0.5559999999999999" rpy="3.141592653589793 -0.0 0.0" />
             <geometry>
                 <mesh filename="../meshes/link1.stl" scale="0.001 0.001 0.001" />
@@ -45,7 +69,7 @@
     <link name="link2">
         <inertial>
-            <origin xyz="-0.0003359368417297048 0.45281365120396316 0.25588731624293615" rpy="0.0 -0.0 0.0" />
+            <origin xyz="-0.0003359368417297048 0.45281365120396344 0.25588731624293615" rpy="0.0 -0.0 0.0" />
             <mass value="1423.0025764040365" />
-            <inertia ixx="327.7826339345211" iyy="38.73396029255571" izz="330.6402748552523" ixy="-0.8519106410419681" iyz="-33.629626749249155" ixz="0.7292926061111302" />
+            <inertia ixx="327.7826339345211" iyy="38.73396029255571" izz="330.64027485525" ixy="-0.8519106410419681" iyz="-33.629626749249155" ixz="0.7292926061111302" />
         </inertial>
         <visual name="link2_visual">
@@ -54,5 +78,5 @@
                 <mesh filename="../meshes/link2.stl" scale="0.001 0.001 0.001" />
             </geometry>
-            <material name="Orange2"/>
+            <material name="Orange1"/>
         </visual>
         <collision name="link2_collision">
@@ -65,7 +89,7 @@
     <link name="link3">
         <inertial>
-            <origin xyz="-0.19088718758387802 0.03189330447130544 0.29068495733124744" rpy="0.0 -0.0 0.0" />
+            <origin xyz="-0.19088718758387802 0.031893304471304874 0.29068495733124744" rpy="0.0 -0.0 0.0" />
             <mass value="1168.7488280092075" />
-            <inertia ixx="39.498903639052514" iyy="171.2938050999797" izz="169.63339154140795" ixy="5.557942574738263" iyz="-1.3072425932029148" ixz="21.704241325588875" />
+            <inertia ixx="39.49890363905433" iyy="171.2938050999797" izz="169.63339154140886" ixy="5.557942574738263" iyz="-1.307242593202929" ixz="21.704241325588875" />
         </inertial>
         <visual name="link3_visual">
@@ -74,5 +98,5 @@
                 <mesh filename="../meshes/link3.stl" scale="0.001 0.001 0.001" />
             </geometry>
-            <material name="Orange2"/>
+            <material name="Orange1"/>
         </visual>
         <collision name="link3_collision">
@@ -87,5 +111,5 @@
             <origin xyz="1.8408047503726266e-06 -0.01046915812392331 -0.2703065523655775" rpy="0.0 -0.0 0.0" />
             <mass value="251.78015853094652" />
-            <inertia ixx="10.075264025066588" iyy="8.082288173467987" izz="4.129550312765559" ixy="-2.604678725859344e-05" iyz="-0.49200640674816576" ixz="-0.00013750705682014086" />
+            <inertia ixx="10.075264025066588" iyy="8.082288173466623" izz="4.129550312764877" ixy="-2.6046787262146154e-05" iyz="-0.49200640674816576" ixz="-0.00013750705670645402" />
         </inertial>
         <visual name="link4_visual">
@@ -94,5 +118,5 @@
                 <mesh filename="../meshes/link4.stl" scale="0.001 0.001 0.001" />
             </geometry>
-            <material name="Orange2"/>
+            <material name="Orange1"/>
         </visual>
         <collision name="link4_collision">
@@ -105,7 +129,7 @@
     <link name="link5">
         <inertial>
-            <origin xyz="0.05215350620219141 2.1698718057905353e-08 -0.13723352234738262" rpy="0.0 -0.0 0.0" />
+            <origin xyz="0.05215350620219141 2.169871777368826e-08 -0.13723352234738262" rpy="0.0 -0.0 0.0" />
             <mass value="142.82201053117632" />
-            <inertia ixx="1.2731956844983188" iyy="2.0365536777011357" izz="1.9890886353753103" ixy="2.871807851079211e-06" iyz="3.614668742102367e-08" ixz="0.3259975845846741" />
+            <inertia ixx="1.273195684498205" iyy="2.0365536777011357" izz="1.989088635375083" ixy="2.871807851079211e-06" iyz="3.614668564466683e-08" ixz="0.3259975845846741" />
         </inertial>
         <visual name="link5_visual">
@@ -127,5 +151,5 @@
             <origin xyz="-5.043046780883742e-07 -1.947194229459104e-06 0.02558859113442196" rpy="0.0 -0.0 0.0" />
             <mass value="14.032085425041553" />
-            <inertia ixx="0.05202564480456573" iyy="0.052026607227617205" izz="0.09842957688901777" ixy="1.8132472401344302e-07" iyz="2.2060905302545564e-07" ixz="3.2715837505747913e-06" />
+            <inertia ixx="0.05202564480456573" iyy="0.05202660722764563" izz="0.09842957688900356" ixy="1.8132472401344302e-07" iyz="2.2060905302545564e-07" ixz="3.2715837505747913e-06" />
         </inertial>
         <visual name="link6_visual">
@@ -143,23 +167,28 @@
         </collision>
     </link>
-    <!--======================= JOINTS =========================-->
-    <joint name="world__base_link" type="fixed">
-        <parent link="world"/>
-        <child link="base_link"/>
-        <origin xyz="0.0 0.0 0.0" rpy="0.0 0.0 0.0"/>
-    </joint>
-    <joint name="base_link_joint_base_link__link1" type="continuous">
-        <origin xyz="0.0 0.0 0.5660000000000001" rpy="3.141592653589793 -0.0 0.0" />
+    <!-- ===================== JOINTS ============================ -->
+    <joint name="world__table" type="fixed">
+        <origin xyz="0.0 0.0 0.0" rpy="0.0 0.0 0.0" />
+        <parent link="world" />
+        <child link="table" />
+    </joint>
+    <joint name="table__base_link" type="fixed">
+        <origin xyz="0.0 0.0 1.206" rpy="0.0 -0.0 0.0" />
+        <parent link="table" />
+        <child link="base_link" />
+    </joint>
+    <joint name="base_link__link1" type="continuous">
+        <origin xyz="0.0 0.0 0.56" rpy="3.141592653589793 -0.0 0.0" />
         <parent link="base_link" />
         <child link="link1" />
         <axis xyz="0.0 0.0 1.0" />
     </joint>
-    <joint name="link1_joint_link1__link2" type="continuous">
-        <origin xyz="0.5 0.064 -0.489" rpy="-1.5707963267948966 -0.0 0.0" />
+    <joint name="link1__link2" type="continuous">
+        <origin xyz="0.5 0.064 -0.48900000000000005" rpy="-1.5707963267948966 -0.0 0.0" />
         <parent link="link1" />
         <child link="link2" />
         <axis xyz="0.0 0.0 1.0" />
     </joint>
-    <joint name="link2_joint_link2__link3" type="continuous">
+    <joint name="link2__link3" type="continuous">
         <origin xyz="0.0 1.3 0.201" rpy="3.141592653589793 -0.0 0.0" />
         <parent link="link2" />
@@ -167,5 +196,5 @@
         <axis xyz="0.0 0.0 1.0" />
     </joint>
-    <joint name="link3_joint_link3__link4" type="continuous">
+    <joint name="link3__link4" type="continuous">
         <origin xyz="0.49900000000000005 0.055 0.255" rpy="1.5707963267948966 -0.0 -1.5707963267948966" />
         <parent link="link3" />
@@ -173,5 +202,5 @@
         <axis xyz="0.0 0.0 1.0" />
     </joint>
-    <joint name="link4_joint_link4__link5" type="continuous">
+    <joint name="link4__link5" type="continuous">
         <origin xyz="0.0 0.165 -0.5359999999999999" rpy="-1.5707963267948966 1.5707963267948966 0" />
         <parent link="link4" />
@@ -179,5 +208,5 @@
         <axis xyz="0.0 0.0 1.0" />
     </joint>
-    <joint name="link5_joint_link5__link6" type="continuous">
+    <joint name="link5__link6" type="continuous">
         <origin xyz="0.2469999999999999 0.0 -0.17500000000000002" rpy="-1.5707963267948966 -0.0 -1.5707963267948966" />
         <parent link="link5" />
@@ -185,5 +214,5 @@
         <axis xyz="0.0 0.0 1.0" />
     </joint>
-    <!--=================== GAZEBO ================-->
+   <!--=================== GAZEBO ================-->
     <material name="Orange1">
         <color rgba="1.0 0.1 0.0 1.0"/>

Commit message: world & models

File: src/kr600/urdf/model.urdf.xacro (robot description, xacro)
@@ -7,12 +7,12 @@
     <link name="table">
         <inertial>
-            <origin xyz="0.0 0.0 0.6" rpy="0.0 0.0 0.0" />
+            <origin xyz="0.0 0.0 0.7" rpy="0.0 0.0 0.0" />
             <mass value="11455.191000000003" />
             <inertia ixx="2543.468607273" iyy="2543.468607273" izz="2310.1301850000045" ixy="-1.4972686767578125e-12" iyz="0.0" ixz="0.0" />
         </inertial>
         <visual name="table_visual">
-            <origin xyz="0.0 0.0 0.6" rpy="0.0 0.0 0.0" />
-            <geometry>
-                <box size="1.1 1.1 1.2" scale="0.001 0.001 0.001"/>
+            <origin xyz="0.0 0.0 0.7" rpy="0.0 0.0 0.0" />
+            <geometry>
+                <box size="1.1 1.1 1.4" scale="0.001 0.001 0.001"/>
                 <!-- <mesh filename="../meshes/table.stl" scale="0.001 0.001 0.001" />> -->
             </geometry>
@@ -20,7 +20,7 @@
         </visual>
         <collision name="table_collision">
-            <origin xyz="0.0 0.0 0.6" rpy="0.0 0.0 0.0" />
-            <geometry>
-                <box size="1.1 1.1 1.2" scale="0.001 0.001 0.001"/>
+            <origin xyz="0.0 0.0 0.7" rpy="0.0 0.0 0.0" />
+            <geometry>
+                <box size="1.1 1.1 1.4" scale="0.001 0.001 0.001"/>
                 <!-- <mesh filename="../meshes/table.stl" scale="0.001 0.001 0.001" /> -->
             </geometry>
@@ -169,5 +169,5 @@
     <!-- ===================== JOINTS ============================ -->
     <joint name="world__table" type="fixed">
-        <origin xyz="0.0 0.0 0.0" rpy="0.0 0.0 0.0" />
+        <origin xyz="0.0 0.0 -0.7" rpy="0.0 0.0 0.0" />
         <parent link="world" />
         <child link="table" />
@@ -222,5 +222,5 @@
     </material>
     <material name="Black">
-        <color rgba="0.1 0.1 0.1 1.0"/>
+        <color rgba="0.05 0.05 0.05 1.0"/>
     </material>
 </robot>

Commit message: aocs_assembly

File: src/kr600/urdf/model.urdf.xacro (robot description, xacro)
@@ -7,12 +7,12 @@
     <link name="table">
         <inertial>
-            <origin xyz="0.0 0.0 0.7" rpy="0.0 0.0 0.0" />
+            <origin xyz="0.0 0.0 0.6" rpy="0.0 0.0 0.0" />
             <mass value="11455.191000000003" />
             <inertia ixx="2543.468607273" iyy="2543.468607273" izz="2310.1301850000045" ixy="-1.4972686767578125e-12" iyz="0.0" ixz="0.0" />
         </inertial>
         <visual name="table_visual">
-            <origin xyz="0.0 0.0 0.7" rpy="0.0 0.0 0.0" />
-            <geometry>
-                <box size="1.1 1.1 1.4" scale="0.001 0.001 0.001"/>
+            <origin xyz="0.0 0.0 0.6" rpy="0.0 0.0 0.0" />
+            <geometry>
+                <box size="1.1 1.1 1.2" scale="0.001 0.001 0.001"/>
                 <!-- <mesh filename="../meshes/table.stl" scale="0.001 0.001 0.001" />> -->
             </geometry>
@@ -20,7 +20,7 @@
         </visual>
         <collision name="table_collision">
-            <origin xyz="0.0 0.0 0.7" rpy="0.0 0.0 0.0" />
-            <geometry>
-                <box size="1.1 1.1 1.4" scale="0.001 0.001 0.001"/>
+            <origin xyz="0.0 0.0 0.6" rpy="0.0 0.0 0.0" />
+            <geometry>
+                <box size="1.1 1.1 1.2" scale="0.001 0.001 0.001"/>
                 <!-- <mesh filename="../meshes/table.stl" scale="0.001 0.001 0.001" /> -->
             </geometry>
@@ -169,5 +169,5 @@
     <!-- ===================== JOINTS ============================ -->
     <joint name="world__table" type="fixed">
-        <origin xyz="0.0 0.0 -0.7" rpy="0.0 0.0 0.0" />
+        <origin xyz="0.0 0.0 -0.6" rpy="0.0 0.0 0.0" />
         <parent link="world" />
         <child link="table" />
