Commit message: kr600_description

File: src/kr600_description/urdf/rviz.urdf.xacro (robot description, xacro)
@@ -1,5 +1,4 @@
 <?xml version="1.0" ?>
 <robot xmlns:xacro="http://wiki.ros.org/xacro" name="kr600">
-<xacro:property name="mesh_path" value="../meshes"/>
    <!-- ===================== links ============================ -->
     <link name="world">
